File: pcb/pcb.kicad_sch (KiCad schematic)
At the start: 281 parts, among them J1 Conn_01x08_Socket, J2 Conn_01x02_Female, U1 YAAJ_WeAct_BlackPill_Part_Lik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

Commit message: Latest updates
Connections:
- net +5V: now also J1.1 (Pin_1); no longer J1.8 (Pin_8)
- net DC: now also J1.5 (Pin_5); no longer J1.4 (Pin_4)
- net GND: now also J1.2 (Pin_2); no longer J1.7 (Pin_7)
- net MOSI_NUM: now also J1.6 (Pin_6); no longer J1.3 (Pin_3)
- net RST: now also J1.4 (Pin_4); no longer J1.5 (Pin_5)
- net SCK_CAPS: now also J1.7 (Pin_7); no longer J1.2 (Pin_2)
- net BL_SOL renamed BL_BUZ
- net BL_BUZ: now also BZ1.1 (-), J1.8 (Pin_8); no longer J1.1 (Pin_1), R4.1
- removed net CS_BUZ: BZ1.1 (-), J1.6 (Pin_6), U1.30 (PA4)
- new net CS_SOL: J1.3 (Pin_3), R4.1, U1.30 (PA4)
Changed lines of the file:
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@@
     (effects (font (size 1.27 1.27)) (justify left bottom))
   )
-  (global_label "CS_BUZ" (shape input) (at 205.105 279.4 180) (fields_autoplaced)
-    (effects (font (size 1.27 1.27)) (justify right))
-    (property "Intersheetrefs" "${INTERSHEET_REFS}" (at 194.8627 279.4 0)
+  (global_label "CS_SOL" (shape input) (at 205.105 279.4 180) (fields_autoplaced)
+    (effects (font (size 1.27 1.27)) (justify right))
+    (property "Intersheetrefs" "${INTERSHEET_REFS}" (at 195.1046 279.4 0)
       (effects (font (size 1.27 1.27)) (justify right) hide)
     )
@@
     )
   )
-  (global_label "BL_SOL" (shape input) (at 81.28 232.41 180) (fields_autoplaced)
-    (effects (font (size 1.27 1.27)) (justify right))
-    (property "Intersheetrefs" "${INTERSHEET_REFS}" (at 71.461 232.41 0)
+  (global_label "BL_BUZ" (shape input) (at 153.035 223.52 180) (fields_autoplaced)
+    (effects (font (size 1.27 1.27)) (justify right))
+    (property "Intersheetrefs" "${INTERSHEET_REFS}" (at 142.9741 223.52 0)
       (effects (font (size 1.27 1.27)) (justify right) hide)
     )
@@
     )
   )
-  (global_label "CS_BUZ" (shape input) (at 153.035 223.52 180) (fields_autoplaced)
-    (effects (font (size 1.27 1.27)) (justify right))
-    (property "Intersheetrefs" "${INTERSHEET_REFS}" (at 142.7927 223.52 0)
+  (global_label "CS_SOL" (shape input) (at 81.28 232.41 180) (fields_autoplaced)
+    (effects (font (size 1.27 1.27)) (justify right))
+    (property "Intersheetrefs" "${INTERSHEET_REFS}" (at 71.2796 232.41 0)
       (effects (font (size 1.27 1.27)) (justify right) hide)
     )
@@
     )
   )
-  (global_label "BL_SOL" (shape input) (at 205.105 266.7 180) (fields_autoplaced)
-    (effects (font (size 1.27 1.27)) (justify right))
-    (property "Intersheetrefs" "${INTERSHEET_REFS}" (at 195.286 266.7 0)
+  (global_label "BL_BUZ" (shape input) (at 205.105 266.7 180) (fields_autoplaced)
+    (effects (font (size 1.27 1.27)) (justify right))
+    (property "Intersheetrefs" "${INTERSHEET_REFS}" (at 195.0441 266.7 0)
       (effects (font (size 1.27 1.27)) (justify right) hide)
     )
@@
     )
   )
-  (global_label "BL_SOL" (shape input) (at 55.88 274.32 180) (fields_autoplaced)
-    (effects (font (size 1.27 1.27)) (justify right))
-    (property "Intersheetrefs" "${INTERSHEET_REFS}" (at 46.061 274.32 0)
+  (global_label "BL_BUZ" (shape input) (at 55.88 274.32 180) (fields_autoplaced)
+    (effects (font (size 1.27 1.27)) (justify right))
+    (property "Intersheetrefs" "${INTERSHEET_REFS}" (at 45.8191 274.32 0)
       (effects (font (size 1.27 1.27)) (justify right) hide)
     )
@@
     )
   )
-  (global_label "CS_BUZ" (shape input) (at 132.08 284.48 0) (fields_autoplaced)
-    (effects (font (size 1.27 1.27)) (justify left))
-    (property "Intersheetrefs" "${INTERSHEET_REFS}" (at 142.3223 284.48 0)
+  (global_label "CS_SOL" (shape input) (at 132.08 284.48 0) (fields_autoplaced)
+    (effects (font (size 1.27 1.27)) (justify left))
+    (property "Intersheetrefs" "${INTERSHEET_REFS}" (at 142.0804 284.48 0)
       (effects (font (size 1.27 1.27)) (justify left) hide)
     )
@@
     )
   )
-  (symbol (lib_id "Connector:Conn_01x08_Socket") (at 210.185 274.32 0) (unit 1)
-    (in_bom yes) (on_board yes) (dnp no) (fields_autoplaced)
-    (property "Reference" "J1" (at 210.8962 274.3779 0)
-      (effects (font (size 1.27 1.27)) (justify left))
-    )
-    (property "Value" "Conn_01x08_Socket" (at 210.8962 276.8021 0)
-      (effects (font (size 1.27 1.27)) (justify left))
-    )
-    (property "Footprint" "" (at 210.185 274.32 0)
-      (effects (font (size 1.27 1.27)) hide)
-    )
-    (property "Datasheet" "~" (at 210.185 274.32 0)
-      (effects (font (size 1.27 1.27)) hide)
-    )
+  (symbol (lib_id "Connector:Conn_01x08_Socket") (at 210.185 276.86 0) (mirror x) (unit 1)
+    (in_bom yes) (on_board yes) (dnp no)
+    (property "Reference" "J1" (at 210.8962 276.8021 0)
+      (effects (font (size 1.27 1.27)) (justify left))
+    )
+    (property "Value" "Conn_01x08_Socket" (at 210.8962 274.3779 0)
+      (effects (font (size 1.27 1.27)) (justify left))
+    )
+    (property "Footprint" "" (at 210.185 276.86 0)
+      (effects (font (size 1.27 1.27)) hide)
+    )
+    (property "Datasheet" "~" (at 210.185 276.86 0)
+      (effects (font (size 1.27 1.27)) hide)
+    )
